File: kicad/light.kicad_sch (KiCad schematic)
At the start: 217 parts, among them J1 USB_C, J2 SM03B-SRSS-TB, J3 Barrell Jack, J4 01x04, J5 Conn_01x09_MountingPin, J6 01x04, J9 Conn_01x09_MountingPin, Q1 NMOS, Q2 NMOS, Q3 NMOS, SW1 Boot, SW2 Reset, SW3 On/Off, SW4 Mode, SW5 RotaryEncoder_Switch_MP, U1 RP2350A-QFN60, U2 TPS5405DR, U3 W25Q128JVS, U4 LBEE5KL1YN-814, U5 TPS2115ADRBR, U6 TPS2115ADRBR, U7 HDC1080, U8 MAX6818EAP_T, U9 PIR223D-S0, Y1 ABM8-272-T3

Commit message: group components
Parts:
- removed TP10: GND, TestPoint:TestPoint_Pad_1.0x1.0mm, symbol Connector:TestPoint
- J8, J9: now not fitted; now left out of the parts list
Changed lines of the file:
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@@
 	)
 	(junction
-		(at 532.13 140.97)
-		(diameter 0)
-		(color 0 0 0 0)
-	)
-	(junction
 		(at 199.39 160.02)
 		(diameter 0)
@@
 	(wire
 		(pts
-			(xy 532.13 138.43) (xy 532.13 140.97)
-		)
-		(stroke
-			(width 0)
-			(type default)
-		)
-	)
-	(wire
-		(pts
 			(xy 359.41 392.43) (xy 382.27 392.43)
 		)
@@
 	(wire
 		(pts
-			(xy 532.13 140.97) (xy 532.13 142.24)
+			(xy 532.13 138.43) (xy 532.13 142.24)
 		)
 		(stroke
@@
 	)
 	(symbol
-		(lib_id "Connector:TestPoint")
-		(at 532.13 140.97 270)
-		(unit 1)
-		(exclude_from_sim no)
-		(in_bom yes)
-		(on_board yes)
-		(dnp no)
-		(property "Reference" "TP10"
-			(at 536.448 139.954 90)
-			(effects
-				(font
-					(size 1.27 1.27)
-				)
-				(justify left)
-			)
-		)
-		(property "Value" "GND"
-			(at 536.702 141.986 90)
-			(effects
-				(font
-					(size 1.27 1.27)
-				)
-				(justify left)
-			)
-		)
-		(property "Footprint" "TestPoint:TestPoint_Pad_1.0x1.0mm"
-			(at 532.13 146.05 0)
-			(effects
-				(font
-					(size 1.27 1.27)
-				)
-				(hide yes)
-			)
-		)
-		(property "Datasheet" "~"
-			(at 532.13 146.05 0)
-			(effects
-				(font
-					(size 1.27 1.27)
-				)
-				(hide yes)
-			)
-		)
-		(property "Description" "test point"
-			(at 532.13 140.97 0)
-			(effects
-				(font
-					(size 1.27 1.27)
-				)
-				(hide yes)
-			)
-		)
-		(pin "1"
-		)
-		(instances
-			(project "light"
-				(path "/fbb17af3-099c-429d-b186-ab4e8e0fdddf"
-					(reference "TP10")
-					(unit 1)
-				)
-			)
-		)
-	)
-	(symbol
 		(lib_id "power:+3V3")
 		(at 317.5 278.13 0)
@@
 		(unit 1)
 		(exclude_from_sim no)
-		(in_bom yes)
+		(in_bom no)
 		(on_board yes)
-		(dnp no)
+		(dnp yes)
 		(property "Reference" "J8"
 			(at 151.13 462.6355 0)
@@
 		(unit 1)
 		(exclude_from_sim no)
-		(in_bom yes)
+		(in_bom no)
 		(on_board yes)
-		(dnp no)
+		(dnp yes)
 		(fields_autoplaced yes)
 		(property "Reference" "J9"

Commit message: general layout
Parts:
- removed JP10: VBUS, Jumper:SolderJumper-2_P1.3mm_Bridged_RoundedPad1.0x1.5mm, symbol Jumper:SolderJumper_2_Bridged
- removed JP11: VREG5, Jumper:SolderJumper-2_P1.3mm_Bridged_RoundedPad1.0x1.5mm, symbol Jumper:SolderJumper_2_Bridged
- removed JP6: 12v in, Jumper:SolderJumper-2_P1.3mm_Bridged_RoundedPad1.0x1.5mm, symbol Jumper:SolderJumper_2_Bridged
- removed JP7: 5v in, Jumper:SolderJumper-2_P1.3mm_Bridged_RoundedPad1.0x1.5mm, symbol Jumper:SolderJumper_2_Bridged
Connections:
- net +12V: now also U6.8 (IN1)
- net +3V3: no longer JP2.1 (A)
- net VBUS: now also U5.8 (IN1)
- net VREG5: now also U5.6 (IN2), U6.6 (IN2)
- net V_RGB: now also J4.4 (Pin_1); no longer J4.1 (Pin_1)
- net at Q1.1 (D): now also J4.3 (Pin_2); no longer J4.2 (Pin_2)
- net at R23.1, U5.1 (STAT): now also JP2.1 (A)
- net at Q3.1 (D): now also J4.1 (Pin_4); no longer J4.4 (Pin_4)
- net at Q2.1 (D): now also J4.2 (Pin_3); no longer J4.3 (Pin_3)
Other:
- moved on the sheet: R23

Commit message: change rgb to 2x4 pins; general layout
Parts:
- removed C40: 1000u, Capacitor_SMD:CP_Elec_8x10, symbol Device:C_Polarized_US
- removed J5: Conn_01x09_MountingPin, Connector_PinSocket_2.54mm:PinSocket_1x09_P2.54mm_Horizontal, symbol Connector_Generic:Conn_01x09
- removed J6: 01x04, Connector_PinSocket_2.54mm:PinSocket_1x04_P2.54mm_Horizontal, symbol Connector_Generic:Conn_01x04
- J4: footprint Connector_PinSocket_2.54mm:PinSocket_1x04_P2.54mm_Horizontal -> Connector_PinSocket_2.54mm:PinSocket_2x04_P2.54mm_Horizontal; symbol Connector_Generic:Conn_01x04 -> Connector_Generic:Conn_02x04_Odd_Even
Connections:
- net ARGB-DATA: now also J4.6 (Pin_4)
- net GND: now also J4.2 (Pin_8)
- net V_RGB: now also J4.7 (Pin_1), J4.8 (Pin_2); no longer J4.4 (Pin_1)
- net at Q1.1 (D): now also J4.5 (Pin_3); no longer J4.3 (Pin_2)
- net at Q2.1 (D): now also J4.3 (Pin_5); no longer J4.2 (Pin_3)
Other:
- note added: "DRGB PWM"
- note added: "RGB"
- note removed: "DRGB PWM step up"
- note removed: "Header pins"
- moved on the sheet: C35, J8, J9
